File: kicad_files/stryx.kicad_sch (KiCad schematic)
At the start: 29 parts, among them J1 Screw_Terminal_M1, J1 USB_B_Micro, J2 Screw_Terminal_M2, J3 Screw_Terminal_Power, SW1 SW_SPDT, U1 LM317_TO-220, U2 NUCLEO-L432KC, U3 TB6612FNG-Module, U4 HC-SR04, U5 NRF24L01_Breakout

Commit message: Set up the footprints
Parts:
- renumbered BT3 to BT1, BT1 to BT3, D4 to D1, D1 to D2, D2 to D3, D3 to D4, D3 to D5, J3 to J1, J1 to J3, J1 to J4, R2 to R1, R1 to R2, U4 to U3, U3 to U4
Changed lines of the file:
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@@
 		(dnp no)
 		(fields_autoplaced yes)
-		(property "Reference" "D3"
+		(property "Reference" "D5"
 			(at 273.05 116.7698 0)
 			(show_name no)
@@
 			(project "stryx"
 				(path "/aa341bb8-bb09-4afa-8a5c-654206316a4d"
-					(reference "D3")
+					(reference "D5")
 					(unit 1)
 				)
@@
 		(dnp no)
 		(fields_autoplaced yes)
-		(property "Reference" "#PWR01"
+		(property "Reference" "#PWR03"
 			(at 83.82 50.8 0)
 			(hide yes)
@@
 			(project "stryx"
 				(path "/aa341bb8-bb09-4afa-8a5c-654206316a4d"
-					(reference "#PWR01")
+					(reference "#PWR03")
 					(unit 1)
 				)
@@
 		(dnp no)
 		(fields_autoplaced yes)
-		(property "Reference" "BT3"
+		(property "Reference" "BT1"
 			(at 25.4 24.7014 0)
 			(show_name no)
@@
 			(project "stryx"
 				(path "/aa341bb8-bb09-4afa-8a5c-654206316a4d"
-					(reference "BT3")
+					(reference "BT1")
 					(unit 1)
 				)
@@
 		(in_pos_files yes)
 		(dnp no)
-		(property "Reference" "U3"
+		(property "Reference" "U4"
 			(at 185.42 22.352 0)
 			(show_name no)
@@
 			(project "stryx"
 				(path "/aa341bb8-bb09-4afa-8a5c-654206316a4d"
-					(reference "U3")
+					(reference "U4")
 					(unit 1)
 				)
@@
 		(dnp no)
 		(fields_autoplaced yes)
-		(property "Reference" "#PWR017"
+		(property "Reference" "#PWR015"
 			(at 252.73 63.5 0)
 			(hide yes)
@@
 			(project "stryx"
 				(path "/aa341bb8-bb09-4afa-8a5c-654206316a4d"
-					(reference "#PWR017")
+					(reference "#PWR015")
 					(unit 1)
 				)
@@
 		(in_pos_files yes)
 		(dnp no)
-		(property "Reference" "#PWR04"
+		(property "Reference" "#PWR012"
 			(at 200.66 31.75 0)
 			(hide yes)
@@
 			(project "stryx"
 				(path "/aa341bb8-bb09-4afa-8a5c-654206316a4d"
-					(reference "#PWR04")
+					(reference "#PWR012")
 					(unit 1)
 				)
@@
 		(dnp no)
 		(fields_autoplaced yes)
-		(property "Reference" "#PWR013"
+		(property "Reference" "#PWR010"
 			(at 162.56 80.01 0)
 			(hide yes)
@@
 			(project "stryx"
 				(path "/aa341bb8-bb09-4afa-8a5c-654206316a4d"
-					(reference "#PWR013")
+					(reference "#PWR010")
 					(unit 1)
 				)
@@
 		(in_pos_files yes)
 		(dnp no)
-		(property "Reference" "#PWR011"
+		(property "Reference" "#PWR017"
 			(at 260.35 137.16 0)
 			(hide yes)
@@
 			(project "stryx"
 				(path "/aa341bb8-bb09-4afa-8a5c-654206316a4d"
-					(reference "#PWR011")
+					(reference "#PWR017")
 					(unit 1)
 				)
@@
 		(in_pos_files yes)
 		(dnp no)
-		(property "Reference" "#PWR018"
+		(property "Reference" "#PWR07"
 			(at 143.51 133.35 0)
 			(hide yes)
@@
 			(project "stryx"
 				(path "/aa341bb8-bb09-4afa-8a5c-654206316a4d"
-					(reference "#PWR018")
+					(reference "#PWR07")
 					(unit 1)
 				)
@@
 		(dnp no)
 		(fields_autoplaced yes)
-		(property "Reference" "D2"
+		(property "Reference" "D3"
 			(at 55.88 87.6299 90)
 			(show_name no)
@@
 			(project "stryx"
 				(path "/aa341bb8-bb09-4afa-8a5c-654206316a4d"
-					(reference "D2")
+					(reference "D3")
 					(unit 1)
 				)
@@
 		(in_pos_files yes)
 		(dnp no)
-		(property "Reference" "#PWR03"
+		(property "Reference" "#PWR011"
 			(at 168.91 35.56 0)
 			(hide yes)
@@
 			(project "stryx"
 				(path "/aa341bb8-bb09-4afa-8a5c-654206316a4d"
-					(reference "#PWR03")
+					(reference "#PWR011")
 					(unit 1)
 				)
@@
 		(dnp no)
 		(fields_autoplaced yes)
-		(property "Reference" "U4"
+		(property "Reference" "U3"
 			(at 181.61 68.5799 0)
 			(show_name no)
@@
 			(project "stryx"
 				(path "/aa341bb8-bb09-4afa-8a5c-654206316a4d"
-					(reference "U4")
+					(reference "U3")
 					(unit 1)
 				)
@@
 		(in_pos_files yes)
 		(dnp no)
-		(property "Reference" "#PWR010"
+		(property "Reference" "#PWR016"
 			(at 260.35 111.76 0)
 			(hide yes)
@@
 			(project "stryx"
 				(path "/aa341bb8-bb09-4afa-8a5c-654206316a4d"
-					(reference "#PWR010")
+					(reference "#PWR016")
 					(unit 1)
 				)
@@
 		(dnp no)
 		(fields_autoplaced yes)
-		(property "Reference" "J1"
+		(property "Reference" "J4"
 			(at 262.89 68.58 0)
 			(show_name no)
@@
 			(project "stryx"
 				(path "/aa341bb8-bb09-4afa-8a5c-654206316a4d"
-					(reference "J1")
+					(reference "J4")
 					(unit 1)
 				)
@@
 		(in_pos_files yes)
 		(dnp no)
-		(property "Reference" "#PWR05"
+		(property "Reference" "#PWR08"
 			(at 157.48 54.61 0)
 			(hide yes)
@@
 			(project "stryx"
 				(path "/aa341bb8-bb09-4afa-8a5c-654206316a4d"
-					(reference "#PWR05")
+					(reference "#PWR08")
 					(unit 1)
 				)
@@
 		(in_pos_files yes)
 		(dnp no)
-		(property "Reference" "#PWR09"
+		(property "Reference" "#PWR06"
 			(at 139.7 130.81 0)
 			(hide yes)
@@
 			(project "stryx"
 				(path "/aa341bb8-bb09-4afa-8a5c-654206316a4d"
-					(reference "#PWR09")
+					(reference "#PWR06")
 					(unit 1)
 				)
@@
 		(dnp no)
 		(fields_autoplaced yes)
-		(property "Reference" "BT1"
+		(property "Reference" "BT3"
 			(at 25.4 39.9414 0)
 			(show_name no)
@@
 			(project "stryx"
 				(path "/aa341bb8-bb09-4afa-8a5c-654206316a4d"
-					(reference "BT1")
+					(reference "BT3")
 					(unit 1)
 				)
@@
 		(in_pos_files yes)
 		(dnp no)
-		(property "Reference" "J1"
+		(property "Reference" "J3"
 			(at 161.036 41.656 0)
 			(show_name no)
@@
 			(project "stryx"
 				(path "/aa341bb8-bb09-4afa-8a5c-654206316a4d"
-					(reference "J1")
+					(reference "J3")
 					(unit 1)
 				)
@@
 		(dnp no)
 		(fields_autoplaced yes)
-		(property "Reference" "#PWR019"
+		(property "Reference" "#PWR014"
 			(at 252.73 29.21 0)
 			(hide yes)
@@
 			(project "stryx"
 				(path "/aa341bb8-bb09-4afa-8a5c-654206316a4d"
-					(reference "#PWR019")
+					(reference "#PWR014")
 					(unit 1)
 				)
@@
 		(dnp no)
 		(fields_autoplaced yes)
-		(property "Reference" "J3"
+		(property "Reference" "J1"
 			(at 97.79 36.83 0)
 			(show_name no)
@@
 			(project "stryx"
 				(path "/aa341bb8-bb09-4afa-8a5c-654206316a4d"
-					(reference "J3")
+					(reference "J1")
 					(unit 1)
 				)
@@
 		(dnp no)
 		(fields_autoplaced yes)
-		(property "Reference" "#PWR012"
+		(property "Reference" "#PWR013"
 			(at 247.65 91.44 0)
 			(hide yes)
@@
 			(project "stryx"
 				(path "/aa341bb8-bb09-4afa-8a5c-654206316a4d"
-					(reference "#PWR012")
+					(reference "#PWR013")
 					(unit 1)
 				)
@@
 		(dnp no)
 		(fields_autoplaced yes)
-		(property "Reference" "R2"
+		(property "Reference" "R1"
 			(at 48.26 99.0599 0)
 			(show_name no)
@@
 			(project "stryx"
 				(path "/aa341bb8-bb09-4afa-8a5c-654206316a4d"
-					(reference "R2")
+					(reference "R1")
 					(unit 1)
 				)
@@
 		(dnp no)
 		(fields_autoplaced yes)
-		(property "Reference" "#PWR015"
+		(property "Reference" "#PWR018"
 			(at 262.89 99.06 0)
 			(hide yes)
@@
 			(project "stryx"
 				(path "/aa341bb8-bb09-4afa-8a5c-654206316a4d"
-					(reference "#PWR015")
+					(reference "#PWR018")
 					(unit 1)
 				)
@@
 		(in_pos_files yes)
 		(dnp no)
-		(property "Reference" "#PWR016"
+		(property "Reference" "#PWR019"
 			(at 271.78 80.01 0)
 			(hide yes)
@@
 			(project "stryx"
 				(path "/aa341bb8-bb09-4afa-8a5c-654206316a4d"
-					(reference "#PWR016")
+					(reference "#PWR019")
 					(unit 1)
 				)
@@
 		(in_pos_files yes)
 		(dnp no)
-		(property "Reference" "#PWR014"
+		(property "Reference" "#PWR09"
 			(at 162.56 69.85 0)
 			(hide yes)
@@
 			(project "stryx"
 				(path "/aa341bb8-bb09-4afa-8a5c-654206316a4d"
-					(reference "#PWR014")
+					(reference "#PWR09")
 					(unit 1)
 				)
@@
 		(dnp no)
 		(fields_autoplaced yes)
-		(property "Reference" "#PWR020"
+		(property "Reference" "#PWR04"
 			(at 102.87 52.07 0)
 			(hide yes)
@@
 			(project "stryx"
 				(path "/aa341bb8-bb09-4afa-8a5c-654206316a4d"
-					(reference "#PWR020")
+					(reference "#PWR04")
 					(unit 1)
 				)
@@
 		(dnp no)
 		(fields_autoplaced yes)
-		(property "Reference" "#PWR07"
+		(property "Reference" "#PWR02"
 			(at 63.5 165.1 0)
 			(hide yes)
@@
 			(project "stryx"
 				(path "/aa341bb8-bb09-4afa-8a5c-654206316a4d"
-					(reference "#PWR07")
+					(reference "#PWR02")
 					(unit 1)
 				)
@@
 		(dnp no)
 		(fields_autoplaced yes)
-		(property "Reference" "D4"
+		(property "Reference" "D1"
 			(at 28.2575 76.2 0)
 			(show_name no)
@@
 			(project "stryx"
 				(path "/aa341bb8-bb09-4afa-8a5c-654206316a4d"
-					(reference "D4")
+					(reference "D1")
 					(unit 1)
 				)
@@
 		(dnp no)
 		(fields_autoplaced yes)
-		(property "Reference" "R1"
+		(property "Reference" "R2"
 			(at 68.58 87.6299 0)
 			(show_name no)
@@
 			(project "stryx"
 				(path "/aa341bb8-bb09-4afa-8a5c-654206316a4d"
-					(reference "R1")
+					(reference "R2")
 					(unit 1)
 				)
@@
 		(dnp no)
 		(fields_autoplaced yes)
-		(property "Reference" "D1"
+		(property "Reference" "D2"
 			(at 45.72 62.23 0)
 			(show_name no)
@@
 			(project "stryx"
 				(path "/aa341bb8-bb09-4afa-8a5c-654206316a4d"
-					(reference "D1")
+					(reference "D2")
 					(unit 1)
 				)
@@
 		(dnp no)
 		(fields_autoplaced yes)
-		(property "Reference" "#PWR02"
+		(property "Reference" "#PWR01"
 			(at 45.72 111.76 0)
 			(hide yes)
@@
 			(project "stryx"
 				(path "/aa341bb8-bb09-4afa-8a5c-654206316a4d"
-					(reference "#PWR02")
+					(reference "#PWR01")
 					(unit 1)
 				)
@@
 		(dnp no)
 		(fields_autoplaced yes)
-		(property "Reference" "D3"
+		(property "Reference" "D4"
 			(at 262.89 110.4899 90)
 			(show_name no)
@@
 			(project "stryx"
 				(path "/aa341bb8-bb09-4afa-8a5c-654206316a4d"
-					(reference "D3")
+					(reference "D4")
 					(unit 1)
 				)
@@
 		(dnp no)
 		(fields_autoplaced yes)
-		(property "Reference" "#PWR06"
+		(property "Reference" "#PWR05"
 			(at 138.43 165.1 0)
 			(hide yes)
@@
 			(project "stryx"
 				(path "/aa341bb8-bb09-4afa-8a5c-654206316a4d"
-					(reference "#PWR06")
+					(reference "#PWR05")
 					(unit 1)
 				)

Commit message: Fixed ultrasonic sensor footprint
Parts:
- U3: footprint XCVR_HC-SR04 -> Connector_PinHeader_1.00mm:PinHeader_1x04_P1.00mm_Vertical
Changed lines of the file:
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@@
 			)
 		)
-		(property "Footprint" "XCVR_HC-SR04"
+		(property "Footprint" "Connector_PinHeader_1.00mm:PinHeader_1x04_P1.00mm_Vertical"
 			(at 167.64 68.58 0)
 			(hide yes)

Commit message: Created Stryx PCB v1
Parts:
- J4: footprint (none) -> Connector_PinHeader_2.54mm:PinHeader_1x05_P2.54mm_Vertical
- U3: footprint Connector_PinHeader_1.00mm:PinHeader_1x04_P1.00mm_Vertical -> Connector_PinHeader_2.54mm:PinHeader_1x04_P2.54mm_Vertical
Changed lines of the file:
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@@
 			)
 		)
-		(property "Footprint" "Connector_PinHeader_1.00mm:PinHeader_1x04_P1.00mm_Vertical"
+		(property "Footprint" "Connector_PinHeader_2.54mm:PinHeader_1x04_P2.54mm_Vertical"
 			(at 167.64 68.58 0)
 			(hide yes)
@@
 			)
 		)
-		(property "Footprint" ""
+		(property "Footprint" "Connector_PinHeader_2.54mm:PinHeader_1x05_P2.54mm_Vertical"
 			(at 266.7 82.55 0)
 			(hide yes)

Commit message: fixed screw terminal footprint
Parts:
- J1, J2, J3: footprint TerminalBlock_MetzConnect:TerminalBlock_MetzConnect_Type703_RT10N02HGLU_1x02_P9.52mm_Horizontal -> TerminalBlock_MetzConnect:TerminalBlock_MetzConnect_Type171_RT13702HBWC_1x02_P7.50mm_Horizontal
Changed lines of the file:
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@@
 			)
 		)
-		(property "Footprint" "TerminalBlock_MetzConnect:TerminalBlock_MetzConnect_Type703_RT10N02HGLU_1x02_P9.52mm_Horizontal"
+		(property "Footprint" "TerminalBlock_MetzConnect:TerminalBlock_MetzConnect_Type171_RT13702HBWC_1x02_P7.50mm_Horizontal"
 			(at 163.83 44.45 0)
 			(hide yes)
@@
 			)
 		)
-		(property "Footprint" "TerminalBlock_MetzConnect:TerminalBlock_MetzConnect_Type703_RT10N02HGLU_1x02_P9.52mm_Horizontal"
+		(property "Footprint" "TerminalBlock_MetzConnect:TerminalBlock_MetzConnect_Type171_RT13702HBWC_1x02_P7.50mm_Horizontal"
 			(at 97.79 45.72 0)
 			(hide yes)
@@
 			)
 		)
-		(property "Footprint" "TerminalBlock_MetzConnect:TerminalBlock_MetzConnect_Type703_RT10N02HGLU_1x02_P9.52mm_Horizontal"
+		(property "Footprint" "TerminalBlock_MetzConnect:TerminalBlock_MetzConnect_Type171_RT13702HBWC_1x02_P7.50mm_Horizontal"
 			(at 163.83 36.83 0)
 			(hide yes)
